Commit message: adding amcl/path_planning to lili_navigation package

File: lili_description/urdf/lili_lidar.urdf.xacro (robot description, xacro)
@@ -8,5 +8,5 @@
       <geometry>
         <!-- dimensions for lidar are rough estimates -->
-        <cylinder length="0.005" radius="0.05" />
+        <cylinder length="0.02" radius="0.05" />
       </geometry>
     </visual>
